File: VICOR.kicad_sch (KiCad schematic)
At the start: 10 parts, among them U7 DCM4623TD2J13D0T00

Commit message: Finished up draft 1 of schematic
Need to look everything over and do a quick layout
Other:
- note added: "DC-DC"
- note removed: "HV->12V DC-DC"
- note removed: "HV-Interface"
- moved on the sheet: C1, C2, C4, F1, L2, L5, R12, R25, R4, U7

Commit message: Started layout
Parts:
- renumbered C4 to C3, L2 to L1, L5 to L2, R12 to R3, R25 to R5, U7 to U1
Changed lines of the file:
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@@
 				)
 				(path "/63c9e8ce-1f6e-4570-90a7-b8c1c309328a/1e68ee3b-d7f5-4ed7-bc45-3e506b43dc1b"
-					(reference "C6")
+					(reference "C4")
 					(unit 1)
 				)
@@
 		(dnp no)
 		(fields_autoplaced yes)
-		(property "Reference" "L5"
+		(property "Reference" "L2"
 			(at 198.12 104.14 90)
 			(show_name no)
@@
 			(project "Blinky"
 				(path "/63c9e8ce-1f6e-4570-90a7-b8c1c309328a/0d1a1f78-7eab-4d69-9e79-2fac59526835"
-					(reference "L5")
-					(unit 1)
-				)
-				(path "/63c9e8ce-1f6e-4570-90a7-b8c1c309328a/1e68ee3b-d7f5-4ed7-bc45-3e506b43dc1b"
-					(reference "L6")
+					(reference "L2")
+					(unit 1)
+				)
+				(path "/63c9e8ce-1f6e-4570-90a7-b8c1c309328a/1e68ee3b-d7f5-4ed7-bc45-3e506b43dc1b"
+					(reference "L4")
 					(unit 1)
 				)
@@
 				)
 				(path "/63c9e8ce-1f6e-4570-90a7-b8c1c309328a/1e68ee3b-d7f5-4ed7-bc45-3e506b43dc1b"
-					(reference "C7")
+					(reference "C5")
 					(unit 1)
 				)
@@
 		(dnp no)
 		(fields_autoplaced yes)
-		(property "Reference" "L2"
+		(property "Reference" "L1"
 			(at 92.71 113.03 90)
 			(show_name no)
@@
 			(project "Blinky"
 				(path "/63c9e8ce-1f6e-4570-90a7-b8c1c309328a/0d1a1f78-7eab-4d69-9e79-2fac59526835"
-					(reference "L2")
+					(reference "L1")
 					(unit 1)
 				)
@@
 		(in_pos_files yes)
 		(dnp no)
-		(property "Reference" "#PWR04"
+		(property "Reference" "#PWR06"
 			(at 163.83 130.81 0)
 			(hide yes)
@@
 			(project "Blinky"
 				(path "/63c9e8ce-1f6e-4570-90a7-b8c1c309328a/0d1a1f78-7eab-4d69-9e79-2fac59526835"
-					(reference "#PWR04")
-					(unit 1)
-				)
-				(path "/63c9e8ce-1f6e-4570-90a7-b8c1c309328a/1e68ee3b-d7f5-4ed7-bc45-3e506b43dc1b"
-					(reference "#PWR010")
+					(reference "#PWR06")
+					(unit 1)
+				)
+				(path "/63c9e8ce-1f6e-4570-90a7-b8c1c309328a/1e68ee3b-d7f5-4ed7-bc45-3e506b43dc1b"
+					(reference "#PWR08")
 					(unit 1)
 				)
@@
 		(in_pos_files yes)
 		(dnp no)
-		(property "Reference" "R25"
+		(property "Reference" "R5"
 			(at 198.12 111.125 90)
 			(show_name no)
@@
 			(project "Blinky"
 				(path "/63c9e8ce-1f6e-4570-90a7-b8c1c309328a/0d1a1f78-7eab-4d69-9e79-2fac59526835"
-					(reference "R25")
-					(unit 1)
-				)
-				(path "/63c9e8ce-1f6e-4570-90a7-b8c1c309328a/1e68ee3b-d7f5-4ed7-bc45-3e506b43dc1b"
-					(reference "R30")
+					(reference "R5")
+					(unit 1)
+				)
+				(path "/63c9e8ce-1f6e-4570-90a7-b8c1c309328a/1e68ee3b-d7f5-4ed7-bc45-3e506b43dc1b"
+					(reference "R8")
 					(unit 1)
 				)
@@
 		(in_pos_files yes)
 		(dnp no)
-		(property "Reference" "C4"
+		(property "Reference" "C3"
 			(at 186.944 119.634 0)
 			(show_name no)
@@
 			(project "Blinky"
 				(path "/63c9e8ce-1f6e-4570-90a7-b8c1c309328a/0d1a1f78-7eab-4d69-9e79-2fac59526835"
-					(reference "C4")
-					(unit 1)
-				)
-				(path "/63c9e8ce-1f6e-4570-90a7-b8c1c309328a/1e68ee3b-d7f5-4ed7-bc45-3e506b43dc1b"
-					(reference "C9")
+					(reference "C3")
+					(unit 1)
+				)
+				(path "/63c9e8ce-1f6e-4570-90a7-b8c1c309328a/1e68ee3b-d7f5-4ed7-bc45-3e506b43dc1b"
+					(reference "C6")
 					(unit 1)
 				)
@@
 		(dnp no)
 		(fields_autoplaced yes)
-		(property "Reference" "U7"
+		(property "Reference" "U1"
 			(at 150.495 104.14 0)
 			(show_name no)
@@
 			(project "Blinky"
 				(path "/63c9e8ce-1f6e-4570-90a7-b8c1c309328a/0d1a1f78-7eab-4d69-9e79-2fac59526835"
-					(reference "U7")
-					(unit 1)
-				)
-				(path "/63c9e8ce-1f6e-4570-90a7-b8c1c309328a/1e68ee3b-d7f5-4ed7-bc45-3e506b43dc1b"
-					(reference "U7")
+					(reference "U1")
+					(unit 1)
+				)
+				(path "/63c9e8ce-1f6e-4570-90a7-b8c1c309328a/1e68ee3b-d7f5-4ed7-bc45-3e506b43dc1b"
+					(reference "U2")
 					(unit 1)
 				)
@@
 		(dnp no)
 		(fields_autoplaced yes)
-		(property "Reference" "#PWR08"
+		(property "Reference" "#PWR07"
 			(at 191.77 130.81 0)
 			(hide yes)
@@
 			(project "Blinky"
 				(path "/63c9e8ce-1f6e-4570-90a7-b8c1c309328a/0d1a1f78-7eab-4d69-9e79-2fac59526835"
-					(reference "#PWR08")
-					(unit 1)
-				)
-				(path "/63c9e8ce-1f6e-4570-90a7-b8c1c309328a/1e68ee3b-d7f5-4ed7-bc45-3e506b43dc1b"
-					(reference "#PWR013")
+					(reference "#PWR07")
+					(unit 1)
+				)
+				(path "/63c9e8ce-1f6e-4570-90a7-b8c1c309328a/1e68ee3b-d7f5-4ed7-bc45-3e506b43dc1b"
+					(reference "#PWR09")
 					(unit 1)
 				)
@@
 				)
 				(path "/63c9e8ce-1f6e-4570-90a7-b8c1c309328a/1e68ee3b-d7f5-4ed7-bc45-3e506b43dc1b"
-					(reference "R14")
+					(reference "R7")
 					(unit 1)
 				)
@@
 		(in_pos_files yes)
 		(dnp no)
-		(property "Reference" "R12"
+		(property "Reference" "R3"
 			(at 88.392 107.95 90)
 			(show_name no)
@@
 			(project "Blinky"
 				(path "/63c9e8ce-1f6e-4570-90a7-b8c1c309328a/0d1a1f78-7eab-4d69-9e79-2fac59526835"
-					(reference "R12")
-					(unit 1)
-				)
-				(path "/63c9e8ce-1f6e-4570-90a7-b8c1c309328a/1e68ee3b-d7f5-4ed7-bc45-3e506b43dc1b"
-					(reference "R13")
-					(unit 1)
-				)
+					(reference "R3")
+					(unit 1)
+				)
+				(path "/63c9e8ce-1f6e-4570-90a7-b8c1c309328a/1e68ee3b-d7f5-4ed7-bc45-3e506b43dc1b"
+					(reference "R6")
+					(unit 1)
+				)

Commit message: Finished layout rev 1
Parts:
- removed F1: 0031.8201, Fuse:Fuseholder_Cylinder-5x20mm_Schurter_0031_8201_Horizontal_Open, symbol AERO_Fuses:Schurter 0031.8201
- added F1: 0031.8221, AERO_Fuses:Schurter 0031.8221, symbol AERO_Fuses:Schurter 0031.8221
Connections:
- net INVERTER+: now also F1.1
- net at L1.1, R3.2: now also F1.2
